File: PPG-Watch.kicad_sch (KiCad schematic)
At the start: 55 parts, among them J1 USB_C_Receptacle_USB2.0_16P, Q1 RE1C002UN, Q2 SI2302CDS, Q3 RE1C002ZP, Q4 RE1C002UN, Q5 RE1C002UN, Q6 RE1C002UN, Q7 RE1C002UN, U1 LSM6DSM, U2 nRF52833_QDxx, U3 MCP73832-2-OT, U4 OPA2381, U5 SR4W035, U6 TPS78227DDC, U7 TXU0101, U8 NJL5821R, U9 TXU0101, Y1 SiT1552

Commit message: Schematic: trans amp ADC IO power
Parts:
- added C15, C17, C18, C19, C20, C21, C23, C24: C, Capacitor_SMD:C_0402_1005Metric, symbol Device:C
- added C22, C25: C, Capacitor_SMD:C_0805_2012Metric, symbol Device:C
- added R15, R16, R17, R18, R19, R20, R21, R22, R23, R24, R25, R26: R, Resistor_SMD:R_0402_1005Metric, symbol Device:R
- added U10: MCP3561R, UQFN20_NC_MCH, symbol Library:MCP3561R
- added U11: MCP23S18x-x-MJ, Package_DFN_QFN:HVQFN-24-1EP_4x4mm_P0.5mm_EP2.6x2.6mm_ThermalVias, symbol Interface_Expansion:MCP23S18x-x-MJ
Connections:
- net +1V8: now also U10.18 (DVDD)
- net +2V7: now also C21.1, R17.2, U10.19 (AVDD)
- net GND: now also D4.10 (PD2_A), D4.2 (PD1_A), C17.2, C18.2, C19.2, C21.2, C23.1, C24.1, R16.1, R21.1, R24.1, U10.17 (DGND), U10.20 (AGND), U10.21 (AGND)
- net USB_D+: now also U2.13 (D+)
- net USB_D-: now also U2.12 (D-)
- net at D4.1 (PD1_C): now also U4.3 (+), C15.1, R15.1
- net at D4.3 (PD2_C): now also U4.5 (+), C20.1, R20.1
- net at U4.1: now also C15.2, R18.1
- net trans_bias: now reaches U4.2 (-)
- net trans_bias: now also U4.6 (-), C18.1, R16.2, R17.1
- net at U4.7: now also C20.2, R19.1
- new net: U10.10 (NC), U10.5 (NC), U10.6 (NC), U10.7 (NC), U10.8 (NC), U10.9 (NC)
- new net: C24.2, R23.1, U10.3 (CH0)
- new net: C23.2, R22.1, U10.4 (CH1)
- new net BB_HPF_out: C22.2, R21.2, R26.1
- new net BB_trans_out: C17.1, C22.1, R15.2, R18.2, R23.2
- new net HPF_bias: R25.2, R26.2
- new net IR_cut_HPF_out: C25.2, R24.2, R25.1
- new net IR_cut_trans_out: C19.1, C25.1, R19.2, R20.2, R22.2
Other:
- note added: "TODO: -IMU -nRF -LED resistors -Level shift en -E-paper power +trans amp +filter -adc -SPI bus"
- note removed: "TODO: IMU nRF LED resistors Level shift en E-paper power trans amp filter adc?"
- moved on the sheet: BT1, C14, C4, C5, C6, C7, C8, D4, J1, L2, Q1, Q3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
