File: PCB_Laser_cut/PPG-Watch.kicad_pcb (KiCad board)
At the start: 2 copper layers, 26.2 x 14.5 mm, 21 parts, among them Q4 RE1C002UN, Q5 RE1C002UN, Q6 RE1C002UN, U4 OPA2381

Commit message: layout complete!!!
Parts:
- removed the REF** at (91.5, 68.4)
- removed the REF** at (91.5, 63.9)
- removed the REF** at (91.5, 59.4)
- added REF**: PinHeader_1x02_P2.54mm_Vertical, Connector_PinHeader_2.54mm:PinHeader_1x02_P2.54mm_Vertical, F.Cu at (115.9, 58.5)
- added REF**: PinHeader_1x05_P2.54mm_Vertical, Connector_PinHeader_2.54mm:PinHeader_1x05_P2.54mm_Vertical, F.Cu at (124.3, 59.1)
- added REF**: PinHeader_1x03_P2.54mm_Vertical, Connector_PinHeader_2.54mm:PinHeader_1x03_P2.54mm_Vertical, F.Cu at (91.0, 61.3)
- added U10: MCP3561R, Package_DFN_QFN:QFN-20-1EP_3x3mm_P0.4mm_EP1.65x1.65mm, F.Cu at (117.5, 64.9)
Routing:
- net /MCLK: track 0.00 -> 7.83 mm
- net /CS3: track 0.00 -> 6.88 mm
- net /PTX: track 0.00 -> 6.56 mm
- net /BB_trans_out: track 6.35 -> 12.7 mm
- net /CLK: track 0.00 -> 5.99 mm
- net /IR_cut_trans_out: track 6.18 -> 12.0 mm
- net /CTX: track 0.00 -> 5.68 mm
- net +1V8: track 0.00 -> 5.28 mm
- net GND: track 3.65 -> 6.60 mm
- net +2V7: track 30.3 -> 29.6 mm
Other:
- board size 26.2 x 14.5 mm -> 38.3 x 15.5 mm
