File: PCB_Laser_cut/PPG-Watch.kicad_sch (KiCad schematic)
At the start: 79 parts, among them J1 USB_C_Receptacle_USB2.0_16P, Q1 RE1C002UN, Q2 SI2302CDS, Q3 RE1C002ZP, Q4 RE1C002UN, Q5 RE1C002UN, Q6 RE1C002UN, Q7 RE1C002UN, U1 LSM6DSM, U10 MCP3561R, U11 MCP23S18x-x-MJ, U2 nRF52833_QDxx, U3 MCP73832-2-OT, U4 OPA2381, U5 SR4W035, U6 TPS78227DDC, U7 TXU0101, U8 NJL5821R, U9 TXU0101, Y1 SiT1552

Commit message: inital component placement
Parts:
- removed U7, U9: TXU0101, Package_SON:Texas_USON-6_1x1.45mm_P0.5mm_SMD, symbol 000_library:TXU0101DRYR
- added C26: 1u, Capacitor_SMD:C_0402_1005Metric, symbol Device:C
- added R27, R28, R29: 0, Resistor_SMD:R_0402_1005Metric, symbol Device:R
- added R30: 10k, Resistor_SMD:R_0402_1005Metric, symbol Device:R
- added U7: TXU0102, Library:X1SON-8_1.05x2mm_P0.5mm, symbol Library:TXU0102DRYR
- C22, C25: value C -> 1u; footprint Capacitor_SMD:C_0805_2012Metric -> Capacitor_SMD:C_0402_1005Metric
- R21, R24, R25, R26: value R -> 0
- U10: footprint UQFN20_NC_MCH -> Package_DFN_QFN:QFN-20-1EP_3x3mm_P0.4mm_EP1.65x1.65mm
Connections:
- net SCL is gone; now on net CLK: DIS1.SCL
- net SDA is gone; now on net CTX: DIS1.SDA
- net +1V8: now also C25.1, R21.1, R25.1, U11.8 (V_{DD}), C26.1, R30.2, U7.7 (VCCB)
- net +2V7: now also C22.2, R26.1, R29.1, U7.3 (VCCA)
- net +BATT: now also R27.1, R28.1
- net BB_HPF_out: no longer C22.2, R21.2, R26.1
- net BB_trans_out: now also R22.2; no longer C22.1, R23.2
- net GND: now also C22.1, C25.2, DIS1.BS1, U1.10 (OCS_Aux), U1.11 (SDO_Aux), U1.2 (SDX), U1.3 (SCX), U11.23 (V_{SS}), C26.2, U7.2 (GND); no longer R21.1, R24.1
- net HPF_bias: no longer R25.2, R26.2
- net IR_cut_HPF_out: no longer C25.2, R24.2, R25.1
- net IR_cut_trans_out: now also R23.2; no longer C25.1, R22.2
- net enc_A: now also U7.8 (B1Y)
- net enc_B: now also U7.1 (B2Y)
- net trans_bias: now also U4.3 (+), U4.5 (+); no longer U4.2 (-), U4.6 (-)
- net CS3: now reaches U10.11 (*CS)
- net CLK: now reaches U10.12 (SCK)
- net CLK: now also U1.13 (SCL), U11.10 (SCK)
- net CTX: now reaches U10.13 (SDI)
- net CTX: now also U1.14 (SDA), U11.11 (SI)
- net PTX: now reaches U10.14 (SDO)
- net PTX: now also U1.1 (SDO/SA0), U11.12 (SO)
- net at U10.15 (*IRQ/MDAT): now also R30.1
- net at C20.1, D4.3 (PD2_C), R20.1: now also U4.2 (-); no longer U4.5 (+)
- net at C20.2, R19.1: now also U4.1; no longer U4.7
- net at DIS1.VCI: now also R24.1, R26.2, R27.2
- net at C13.2, DIS1.VDD: now also R21.2
- net at DIS1.VDDIO: now also R24.2, R25.2
- net CS2: now reaches U1.12 (CS)
- net IMU_int1: now reaches U1.4 (INT1)
- net IMU_int2: now reaches U1.9 (INT2)
- net at C15.2, R18.1: now also U4.7; no longer U4.1
- net at C15.1, D4.1 (PD1_C), R15.1: now also U4.6 (-); no longer U4.3 (+)
- net at U8.3 (B): now also U7.4 (A2)
- net at U8.4 (A): now also U7.5 (A1)
- net CS4: now reaches U11.9 (~{CS})
- net at C1.1, L1.1: now also R28.2, R29.2
- net CS renamed CS1
- new net enc_en: U7.6 (OE)
- no-connect marks 5 -> 9
Other:
- note added: "TODO: +IMU -nRF +E-paper power +trans amp +filter +adc -SPI bus -check CTX for 3-wire -LED resistors -Filters"
- note removed: "TODO: -IMU -nRF -LED resistors -Level shift en -E-paper power +trans amp +filter -adc -SPI bus"
- moved on the sheet: C10, C12, C13, C14, C23, C24, C6, C7, C8, L2, R22, R23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

Commit message: layout complete!!!
Parts:
- removed BT1: Battery, symbol Device:Battery
- removed C1, C2, C4, C5: 4u7, Capacitor_SMD:C_0805_2012Metric, symbol Device:C
- removed C10, C11, C12, C13, C16, C3, C9: 1u, Capacitor_SMD:C_0805_2012Metric, symbol Device:C
- removed C14, C18, C21, C23, C24, C8: C, Capacitor_SMD:C_0402_1005Metric, symbol Device:C
- removed C22, C25, C26, C6, C7: 1u, Capacitor_SMD:C_0402_1005Metric, symbol Device:C
- removed D1, D2, D3: CTS05S30, E-Paper_Watch-Library:D_SOD-882, symbol Device:D
- removed DIS1: GDEH0154D67, E-Paper_Watch-Library:GDEH0154D67, symbol E-Paper-Watch-Library:GDEH0154D67
- removed J1: USB_C_Receptacle_USB2.0_16P, Library:GCT_USB4720-03-A_REVA, symbol Connector:USB_C_Receptacle_USB2.0_16P
- removed L1: 47u, Inductor_SMD:L_Bourns-SRN4018, symbol Device:L_Iron
- removed L2: L, Inductor_SMD:L_0402_1005Metric, symbol Device:L
- removed Q1, Q7: RE1C002UN, Package_TO_SOT_SMD:SOT-416, symbol Transistor_FET:Q_NMOS_GSD
- removed Q2: SI2302CDS, Package_TO_SOT_SMD:SOT-23, symbol Transistor_FET:DMN2230U
- removed Q3: RE1C002ZP, Package_TO_SOT_SMD:SOT-416, symbol Transistor_FET:Q_PMOS_GSD
- removed R1, R4, R6: 1M, Resistor_SMD:R_0402_1005Metric, symbol Device:R
- removed R14, R16, R17, R22, R23: R, Resistor_SMD:R_0402_1005Metric, symbol Device:R
- removed R2: 1M5, Resistor_SMD:R_0402_1005Metric, symbol Device:R
- removed R21, R24, R25, R26, R27, R28, R29: 0, Resistor_SMD:R_0402_1005Metric, symbol Device:R
- removed R3: 2R2, Resistor_SMD:R_0402_1005Metric, symbol Device:R
- removed R5: 220k, Resistor_SMD:R_0402_1005Metric, symbol Device:R
- removed R7, R8: 5k1, Resistor_SMD:R_0402_1005Metric, symbol Device:R
- removed R9: 2k2, Resistor_SMD:R_0402_1005Metric, symbol Device:R
- removed U1: LSM6DSM, Package_LGA:LGA-14_3x2.5mm_P0.5mm_LayoutBorder3x4y, symbol Sensor_Motion:LSM6DSM
- removed U11: MCP23S18x-x-MJ, Package_DFN_QFN:HVQFN-24-1EP_4x4mm_P0.5mm_EP2.6x2.6mm_ThermalVias, symbol Interface_Expansion:MCP23S18x-x-MJ
- removed U2: nRF52833_QDxx, Package_DFN_QFN:QFN-40-1EP_5x5mm_P0.4mm_EP3.6x3.6mm, symbol MCU_Nordic:nRF52833_QDxx
- removed U3: MCP73832-2-OT, Package_TO_SOT_SMD:SOT-23-5, symbol Battery_Management:MCP73832-2-OT
- removed U5: SR4W035, Library:SR4W035_4X6_ANT, symbol 000_library:SR4W035
- removed U6: TPS78227DDC, Package_TO_SOT_SMD:SOT-23-5, symbol Regulator_Linear:TPS78227DDC
- removed U7: TXU0102, Library:X1SON-8_1.05x2mm_P0.5mm, symbol Library:TXU0102DRYR
- removed U8: NJL5821R, Library:NJL5821R, symbol 000_library:NJL5821R
- removed Y1: SiT1552, Library:SiT1552, symbol 000_library:SiT1552
Connections:
- net trans_bias is gone; now on net GND: U4.3 (+), U4.5 (+)
- net BB_trans_out: now also U10.4 (CH1)
- net IR_cut_trans_out: now also U10.3 (CH0)
- net MCLK: now reaches U10.16 (MCLK)
- no-connect marks 9 -> 2
Other:
- note removed: "TODO: +IMU -nRF +E-paper power +trans amp +filter +adc -SPI bus -check CTX for 3-wire -LED resistors -Filters"
- moved on the sheet: R30
