File: PCB/PPG-Watch.kicad_sch (KiCad schematic)
At the start: 79 parts, among them J1 USB_C_Receptacle_USB2.0_16P, Q1 RE1C002UN, Q2 SI2302CDS, Q3 RE1C002ZP, Q4 RE1C002UN, Q5 RE1C002UN, Q6 RE1C002UN, Q7 RE1C002UN, U1 LSM6DSM, U10 MCP3561R, U11 MCP23S18x-x-MJ, U2 nRF52833_QDxx, U3 MCP73832-2-OT, U4 OPA2381, U5 SR4W035, U6 TPS78227DDC, U7 TXU0102, U8 NJL5821R, Y1 SiT1552

Commit message: layout complete!!!
Parts:
- added C23, C32: 1u, Capacitor_SMD:C_0402_1005Metric, symbol Device:C
- added C28, C29: 100n, Capacitor_SMD:C_0402_1005Metric, symbol Device:C
- added C30: 100p, Capacitor_SMD:C_0402_1005Metric, symbol Device:C
- added C31: 47n, Capacitor_SMD:C_0402_1005Metric, symbol Device:C
- added J2: Conn_ARM_SWD_TagConnect_TC2030-NL, Connector:Tag-Connect_TC2030-IDC-NL_2x03_P1.27mm_Vertical, symbol Connector:Conn_ARM_SWD_TagConnect_TC2030-NL
- added L3: 10u, Inductor_SMD:L_0603_1608Metric, symbol Device:L
- added L4: 15n, Inductor_SMD:L_0402_1005Metric, symbol Device:L
- BT1: footprint Connector_PinHeader_2.54mm:PinHeader_1x02_P2.54mm_Vertical -> Library:Battery
- C14: value C -> 1p2
- C8: value C -> 1p5
- L2: value L -> 4n2
Connections:
- net enc_en is gone; now on net +2V7: U7.6 (OE)
- net +1V8: now also U11.13 (~{RESET}), C28.1, J2.1 (VCC)
- net 2V7_en: now also U11.3 (GPB3)
- net BUSY: now also U11.22 (GPA7)
- net CLK: now also U2.36 (AIN7/P0.31)
- net CS1: now also U2.33 (AIN4/P0.28)
- net CS2: now also U2.17 (P0.20)
- net CS3: now also U2.34 (AIN5/P0.29)
- net CS4: now also U2.32 (AIN0/P0.02)
- net CTX: now also U2.14 (P0.15)
- net D/C: now also U2.35 (AIN6/P0.30)
- net GLED_en: now also U11.2 (GPB2)
- net GND: now also DIS1.GND1, DIS1.GND2, C23.1, C28.2, C29.1, C30.1, C31.2, C32.2, J2.5 (GND)
- net IMU_int1: now also U2.7 (P0.11)
- net IMU_int2: now also U2.6 (P1.09)
- net IRLED_en: now also U11.6 (GPB6)
- net PTX: now also U2.15 (P0.17)
- net RES: now also U11.21 (GPA6)
- net RLED_en: now also U11.7 (GPB7)
- net bat_mon: now also U2.5 (AIN3/P0.05)
- net bat_mon_en: now also U11.4 (GPB4)
- net charge_stat: now also U11.5 (GPB5)
- net enc_A: now also U11.1 (GPB1)
- net enc_B: now also U11.24 (GPB0)
- net enc_LED_en: now also U11.18 (GPA3)
- net at U2.1 (DEC1): now also C29.2
- net at U2.11 (DECUSB): now also C23.2
- net at U2.16 (P0.18/~{RESET}): now also J2.3 (~{RESET})
- net at U2.19 (SWDIO): now also J2.2 (SWDIO)
- net at U2.20 (SWDCLK): now also J2.4 (SWCLK)
- net at U2.26 (DEC6): now also U2.38 (DEC4), C31.1, C32.1, L4.1
- net at U2.27 (DEC3): now also C30.2
- net Int: now reaches U2.31 (AIN1/P0.03)
- net Int: now also U11.14 (INTA)
- net at U2.39 (DCC): now also L3.2
- net MCLK: now reaches U2.4 (AIN2/P0.04)
- net MCLK: now also U10.16 (MCLK)
- new net: L3.1, L4.2
- no-connect marks 9 -> 12
Other:
- note added: "2.7V regulator"
- note added: "Analog Front End"
- note added: "Battery"
- note added: "Display"
- note added: "Encoder"
- note added: "IMU"
- note added: "IO Expander"
- note added: "TODO: +IMU +nRF +E-paper power +trans amp +filter +adc +SPI bus +check CTX for 3-wire -LED resistors -Filters"
- note added: "USB-C"
- note added: "nRF52833"
- note removed: "TODO: +IMU -nRF +E-paper power +trans amp +filter +adc -SPI bus -check CTX for 3-wire -LED resistors -Filters"
- moved on the sheet: BT1, C1, C10, C11, C12, C13, C14, C15, C16, C17, C18, C19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

Commit message: board ordered!!!
Parts:
- added J3: Conn_01x02_Pin, Connector_PinSocket_1.00mm:PinSocket_1x02_P1.00mm_Vertical, symbol Connector:Conn_01x02_Pin
Connections:
- net +1V8: now also U1.10 (OCS_Aux), U1.11 (SDO_Aux), U1.2 (SDX), U1.3 (SCX)
- net +BATT: now also Q3.2 (S); no longer Q3.3 (D)
- net GND: no longer U1.10 (OCS_Aux), U1.11 (SDO_Aux), U1.2 (SDX), U1.3 (SCX)
- net NFC1: now reaches U2.22 (NFC1/P0.09)
- net NFC1: now also J3.2 (Pin_2)
- net NFC2: now reaches U2.23 (NFC2/P0.10)
- net NFC2: now also J3.1 (Pin_1)
- net at R2.1: now also Q3.3 (D); no longer Q3.2 (S)
- net Int renamed IO_INT
Other:
- note added: "TODO: -LED resistors -Filters"
- note removed: "TODO: +IMU +nRF +E-paper power +trans amp +filter +adc +SPI bus +check CTX for 3-wire -LED resistors -Filters"
- title: (none) -> PPG Watch
- moved on the sheet: C16, C18, Q4, Q5, Q6, R16, R17
